File: Hardware/Design/PCB-DRV/PCB-DRV.kicad_pcb (KiCad board)
At the start: 2 copper layers, 80 x 80 mm, 26 parts, among them J1 STEP_MX, J2 MCU_STEP/DIR, J3 MCU_EN&UART, J4 VIO&VM, J5 STEP_MY, J6 STEP_MZ, U1 TMC2209_SILENTSTEPSTICK, U2 TMC2209_SILENTSTEPSTICK, U3 TMC2209_SILENTSTEPSTICK

Commit message: FIX del pin 12 al pin 13 para driver V985, movi la alimentación a separada, 12V y 3.3V, hice un selector de driver o tipo de driver
Parts:
- removed R1: 1K, Resistor_THT:R_Axial_DIN0309_L9.0mm_D3.2mm_P12.70mm_Horizontal
- added J7: +12V, TerminalBlock_Phoenix:TerminalBlock_Phoenix_MKDS-1,5-2-5.08_1x02_P5.08mm_Horizontal, F.Cu at (61.0, 5.50)
- added J8: UART_CONF, Connector_PinHeader_2.54mm:PinHeader_1x03_P2.54mm_Vertical, F.Cu at (53.3, 58.8)
- J4: value VIO&VM -> +3.3V; footprint Connector_JST:JST_XH_B3B-XH-A_1x03_P2.50mm_Vertical -> Connector_JST:JST_XH_B2B-XH-A_1x02_P2.50mm_Vertical
- moved R3 5.50 mm to (63.5, 67.8)
- moved J4 5.39 mm to (41.0, 4.00), turned to 0 degrees
- moved R2 5.00 mm to (44.0, 67.8)
Connections:
- J3 pad 2: /GPIO_UART -> GPIO_UART
- U1 pad 12: GPIO_UART -> GPIO_UART_SLNK
- U1 pad 13: unconnected-(U1-SPRD-Pad13) -> GPIO_UART_V985
- U2 pad 12: GPIO_UART -> GPIO_UART_SLNK
- U2 pad 13: unconnected-(U2-SPRD-Pad13) -> GPIO_UART_V985
- U3 pad 12: GPIO_UART -> GPIO_UART_SLNK
- U3 pad 13: unconnected-(U3-SPRD-Pad13) -> GPIO_UART_V985
Routing:
- net GPIO_UART_SLNK: track 0.00 -> 210.6 mm
- net GPIO_UART_V985: track 0.00 -> 151.1 mm
- net GPIO_UART: track 139.8 -> 14.1 mm
- net +12V: track 137.9 -> 159.0 mm
- net GPIO_EN_Z: track 80.9 -> 87.5 mm
- net /GPIO_UART: track 4.15 -> 0.00 mm
- net +3.3V: track 206.5 -> 207.8 mm
Other:
- board text added: "+"
- board text added: "-"
- board text added: "PCB-DRV-V2"
- board text removed: "AT_Drivers_V1"
