File: Hardware/Design/PCB-DRV/PCB-DRV.kicad_sch (KiCad schematic)
At the start: 21 parts, among them J1 STEP_MX, J2 MCU_STEP/DIR, J3 MCU_EN&UART, J4 VIO&VM, J5 STEP_MY, J6 STEP_MZ, U1 TMC2209_SILENTSTEPSTICK, U2 TMC2209_SILENTSTEPSTICK, U3 TMC2209_SILENTSTEPSTICK

Commit message: FIX del pin 12 al pin 13 para driver V985, movi la alimentación a separada, 12V y 3.3V, hice un selector de driver o tipo de driver
Parts:
- removed J4: VIO&VM, Connector_JST:JST_XH_B3B-XH-A_1x03_P2.50mm_Vertical, symbol Connector_Generic:Conn_01x03
- removed R1: 1K, Resistor_THT:R_Axial_DIN0309_L9.0mm_D3.2mm_P12.70mm_Horizontal, symbol Device:R
- added J4: +3.3V, Connector_JST:JST_XH_B2B-XH-A_1x02_P2.50mm_Vertical, symbol Connector_Generic:Conn_01x02
- added J7: +12V, TerminalBlock_Phoenix:TerminalBlock_Phoenix_MKDS-1,5-2-5.08_1x02_P5.08mm_Horizontal, symbol Connector_Generic:Conn_01x02
- added J8: UART_CONF, Connector_PinHeader_2.54mm:PinHeader_1x03_P2.54mm_Vertical, symbol Connector_Generic:Conn_01x03
Connections:
- net /GPIO_UART is gone; now on net GPIO_UART: J3.2 (Pin_2)
- net +12V: now also J7.1 (Pin_1)
- net +3.3V: now also J4.1 (Pin_1)
- net GND: now also J4.2 (Pin_2), J7.2 (Pin_2)
- net GPIO_UART: now also J8.2 (Pin_2); no longer U1.12 (UART), U2.12 (UART), U3.12 (UART)
- net GPIO_UART_V985: now reaches U2.13 (SPRD)
- net GPIO_UART_V985: now also U1.13 (SPRD), U3.13 (SPRD), J8.1 (Pin_1)
- new net GPIO_UART_SLNK: J8.3 (Pin_3), U1.12 (UART), U2.12 (UART), U3.12 (UART)
Other:
- note added: "Si usas TMC 2209 V985 el puente va entre pin 2 Y 1 Si usas TMC 2209 de SilentStepStick el puente va entre pin 2 Y 3"
