File: Hardware/Design/PCB-HUS/PCB-HUS.kicad_sch (KiCad schematic)
At the start: 10 parts, among them J1 MOTOR, J2 GND_STAR, J3 GPIO_MCU, J4 VMOT, Q1 IRLZ24, U1 PC817

Commit message: reubicación del errata. Cambio en el contenido de readme. Agregue el Firmware de fluid NC
Connections:
- net GPIO4_ESP32 renamed PWM
Changed lines of the file:
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@@
 		)
 	)
-	(global_label "GPIO4_ESP32"
+	(global_label "PWM"
 		(shape input)
 		(at 30.48 25.4 0)
@@
 		)
 		(property "Intersheetrefs" "${INTERSHEET_REFS}"
-			(at 46.1651 25.4 0)
+			(at 37.638 25.4 0)
 			(hide yes)
 			(show_name no)
@@
 		)
 	)
-	(global_label "GPIO4_ESP32"
+	(global_label "PWM"
 		(shape output)
 		(at 106.68 25.4 180)
@@
 		)
 		(property "Intersheetrefs" "${INTERSHEET_REFS}"
-			(at 90.9949 25.4 0)
+			(at 99.522 25.4 0)
 			(hide yes)
 			(show_name no)
@@
 		)
 		(instances
-			(project "PCB-HUS-V1"
+			(project "PCB-HUS"
 				(path "/2ec725a5-f70e-4f0c-8c57-7d4984c09f68"
 					(reference "R1")
@@
 		)
 		(instances
-			(project "PCB-HUS-V1"
+			(project "PCB-HUS"
 				(path "/2ec725a5-f70e-4f0c-8c57-7d4984c09f68"
 					(reference "J3")
@@
 		)
 		(instances
-			(project "PCB-HUS-V1"
+			(project "PCB-HUS"
 				(path "/2ec725a5-f70e-4f0c-8c57-7d4984c09f68"
 					(reference "#PWR04")
@@
 		)
 		(instances
-			(project "PCB-HUS-V1"
+			(project "PCB-HUS"
 				(path "/2ec725a5-f70e-4f0c-8c57-7d4984c09f68"
 					(reference "#PWR03")
@@
 		)
 		(instances
-			(project "PCB-HUS-V1"
+			(project "PCB-HUS"
 				(path "/2ec725a5-f70e-4f0c-8c57-7d4984c09f68"
 					(reference "#PWR02")
@@
 		)
 		(instances
-			(project "PCB-HUS-V1"
+			(project "PCB-HUS"
 				(path "/2ec725a5-f70e-4f0c-8c57-7d4984c09f68"
 					(reference "J4")
@@
 		)
 		(instances
-			(project "PCB-HUS-V1"
+			(project "PCB-HUS"
 				(path "/2ec725a5-f70e-4f0c-8c57-7d4984c09f68"
 					(reference "J2")
@@
 		)
 		(instances
-			(project "PCB-HUS-V1"
+			(project "PCB-HUS"
 				(path "/2ec725a5-f70e-4f0c-8c57-7d4984c09f68"
 					(reference "Q1")
@@
 		)
 		(instances
-			(project "PCB-HUS-V1"
+			(project "PCB-HUS"
 				(path "/2ec725a5-f70e-4f0c-8c57-7d4984c09f68"
 					(reference "R2")
@@
 		)
 		(instances
-			(project "PCB-HUS-V1"
+			(project "PCB-HUS"
 				(path "/2ec725a5-f70e-4f0c-8c57-7d4984c09f68"
 					(reference "J1")
@@
 		)
 		(instances
-			(project "PCB-HUS-V1"
+			(project "PCB-HUS"
 				(path "/2ec725a5-f70e-4f0c-8c57-7d4984c09f68"
 					(reference "#PWR06")
@@
 		)
 		(instances
-			(project "PCB-HUS-V1"
+			(project "PCB-HUS"
 				(path "/2ec725a5-f70e-4f0c-8c57-7d4984c09f68"
 					(reference "R3")
@@
 		)
 		(instances
-			(project "PCB-HUS-V1"
+			(project "PCB-HUS"
 				(path "/2ec725a5-f70e-4f0c-8c57-7d4984c09f68"
 					(reference "D1")
@@
 		)
 		(instances
-			(project "PCB-HUS-V1"
+			(project "PCB-HUS"
 				(path "/2ec725a5-f70e-4f0c-8c57-7d4984c09f68"
 					(reference "U1")
@@
 		)
 		(instances
-			(project "PCB-HUS-V1"
+			(project "PCB-HUS"
 				(path "/2ec725a5-f70e-4f0c-8c57-7d4984c09f68"
 					(reference "#PWR05")
@@
 		)
 		(instances
-			(project "PCB-HUS-V1"
+			(project "PCB-HUS"
 				(path "/2ec725a5-f70e-4f0c-8c57-7d4984c09f68"
 					(reference "#PWR01")
